File: schematic/BLDC_Proto.kicad_pcb (KiCad board)
At the start: 2 copper layers, 150 x 100 mm, 50 parts, among them J1 Motor Encoder In, M1 Hobbywing QuicRun 3650, Q1 GSFN0390, Q2 GSFN0390, Q3 GSFN0390, Q4 GSFN0390, Q5 GSFN0390, Q6 GSFN0390, SW1 SW_Push, SW2 Keypad, U1 ESP32-S3-DevKitC, U2 AP62200TWU, U3 DRV8300D, U4 74HC595, U5 74HC595, U6 BA56-12SURKWA, U7 BA56-12SURKWA

Commit message: 2nd iteration
Parts:
- removed M1: Hobbywing QuicRun 3650, footprints:BLDC
- removed R14, R15, R16, R17, R18: 680, Resistor_SMD:R_0805_2012Metric
- removed U5: 74HC595, Package_SO:TSSOP-16_4.4x5mm_P0.65mm
- removed U6, U7: BA56-12SURKWA, footprints:BA56-12SURKWA
- added C12: 1uF, Capacitor_SMD:C_0805_2012Metric, B.Cu at (89.8, 116.0)
- added C13: 1uF, Capacitor_SMD:C_0805_2012Metric, F.Cu at (90.8, 119.0)
- added C14: 22uF, Capacitor_SMD:C_1210_3225Metric, F.Cu at (96.2, 124.2)
- added C15: 1mF, Capacitor_THT:CP_Radial_D13.0mm_P5.00mm, F.Cu at (88.8, 137.8)
- added C16: 100nF, Capacitor_SMD:C_0805_2012Metric, F.Cu at (103.2, 154.8)
- added C17: 22uF, Capacitor_SMD:C_1210_3225Metric, F.Cu at (108.0, 153.5)
- added C18: 22uF, Capacitor_SMD:C_1210_3225Metric, F.Cu at (108.0, 157.0)
- added C19: 10uF, Capacitor_SMD:C_1206_3216Metric, F.Cu at (95.5, 157.0)
- added D2: MMSZ5245B, Diode_SMD:D_SOD-123, B.Cu at (81.8, 130.0)
- added D3: MMSZ5245B, Diode_SMD:D_SOD-123, B.Cu at (81.8, 135.8)
- added D4: MMSZ5245B, Diode_SMD:D_SOD-123, B.Cu at (81.8, 118.0)
- added D5: MMSZ5245B, Diode_SMD:D_SOD-123, B.Cu at (81.8, 123.8)
- added D6: MMSZ5245B, Diode_SMD:D_SOD-123, B.Cu at (92.8, 118.5)
- added D7: MMSZ5245B, Diode_SMD:D_SOD-123, B.Cu at (87.0, 118.5)
- added D8: SMCJ15A, Diode_SMD:D_SMC, B.Cu at (80.0, 144.0)
- added D9: SB2060, Diode_THT:D_DO-201AD_P15.24mm_Horizontal, F.Cu at (72.4, 151.5)
- added M1A: TestPoint, footprints:TestPoint_THTPad_D5.0mm_Drill3.0mm, F.Cu at (73.0, 133.0)
- added M1B: TestPoint, footprints:TestPoint_THTPad_D5.0mm_Drill3.0mm, F.Cu at (73.0, 120.8)
- added M1C: TestPoint, footprints:TestPoint_THTPad_D5.0mm_Drill3.0mm, F.Cu at (90.0, 109.8)
- C1: value 10uF -> 1uF; footprint Capacitor_SMD:C_1206_3216Metric -> Capacitor_SMD:C_0805_2012Metric
- C11, C5, C7, C8: moved to B.Cu
- C2: value 330nF -> 1uF
- C3, C9: value 22uF -> 1uF; footprint Capacitor_SMD:C_1210_3225Metric -> Capacitor_SMD:C_0805_2012Metric
- C4: value 22uF -> 1uF; footprint Capacitor_SMD:C_1210_3225Metric -> Capacitor_SMD:C_0805_2012Metric; moved to B.Cu
- L1: value 4.7uH -> 15uH; footprint footprints:Inductor_2424 -> footprints:HCM1A0805V3-150R
- Q1, Q2, Q3, Q4, Q5, Q6: value GSFN0390 -> GSFN6982
- R1: value 56.2k -> 4.7k
- R11: value 680 -> 24k
- R12: value 680 -> 100k
- R13: value 680 -> 3k
- R2: value 10k -> 4.7k
- R3, R4: value 10k -> 15
- R5, R6: value 15 -> 10k
- U1: value ESP32-S3-DevKitC -> NHD-C0220BIZ; footprint PCM_Espressif:ESP32-S3-DevKitC -> Display:NHD-C0220BiZ
- U2: value AP62200TWU -> DRV8300D; footprint Package_TO_SOT_SMD:TSOT-23-6 -> Package_SO:TSSOP-20_4.4x6.5mm_P0.65mm
- U3: value DRV8300D -> ESP32-S3-DevKitC; footprint Package_SO:TSSOP-20_4.4x6.5mm_P0.65mm -> PCM_Espressif:ESP32-S3-DevKitC
- U4: value 74HC595 -> TPP302080; footprint Package_SO:TSSOP-16_4.4x5mm_P0.65mm -> Package_TO_SOT_SMD:TSOT-23-6
- moved C5 121.8 mm to (77.2, 132.5), turned to -90 degrees
- moved R3 120.3 mm to (82.2, 129.8), turned to 180 degrees
- moved R5 118.4 mm to (203.2, 139.2), turned to -90 degrees
- moved R4 116.8 mm to (82.2, 134.2)
- moved R6 115.1 mm to (199.8, 143.0)
- moved C1 103.0 mm to (182.5, 90.8), turned to 0 degrees
- moved R12 102.9 mm to (103.8, 157.8), turned to 180 degrees
- moved R11 101.2 mm to (102.5, 160.5), turned to 180 degrees
- moved C9 100.5 mm to (199.0, 146.2)
- moved R13 99.5 mm to (98.8, 160.5), turned to 180 degrees
- moved R1 93.9 mm to (175.2, 91.8)
- moved R2 92.1 mm to (177.5, 91.8), turned to 90 degrees
- moved C11 91.2 mm to (89.8, 114.0), turned to 180 degrees
- moved U4 86.9 mm to (99.8, 157.0), turned to 0 degrees
- moved C10 86.2 mm to (82.2, 120.0), turned to 180 degrees
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Connections:
- C1 pad 1: +12V -> +3.3V
- C10 pad 1: GND -> Net-(U2-BSTB)
- C10 pad 2: +3.3V -> Net-(D4-A)
- C11 pad 1: GND -> +12V
- C11 pad 2: +3.3V -> GND
- C2 pad 1: Net-(U2-SW) -> +3.3V
- C2 pad 2: Net-(U2-BST) -> Net-(U1-VOUT)
- C3 pad 1: +5V -> Net-(U1-C1+)
- C3 pad 2: GND -> Net-(U1-C1-)
- C4 pad 1: +5V -> +12V
- C5 pad 1: Net-(U1-GPIO8/ADC1_CH7) -> +12V
- C6 pad 1: Net-(U3-BSTA) -> Net-(U2-BSTA)
- C6 pad 2: Net-(M1-A) -> Net-(D2-A)
- C7 pad 1: Net-(U3-BSTB) -> +12V
- C7 pad 2: Net-(M1-B) -> GND
- C8 pad 1: Net-(U3-BSTC) -> +12V
- C8 pad 2: Net-(M1-C) -> GND
- C9 pad 1: GND -> Net-(U3-GPIO8/ADC1_CH7)
- C9 pad 2: +12V -> GND
- L1 pad 1: Net-(U2-SW) -> Net-(U4-SW)
- Q1 pad 1: Net-(M1-A) -> Net-(D2-A)
- Q1 pad 2: Net-(M1-A) -> Net-(D2-A)
- Q1 pad 3: Net-(M1-A) -> Net-(D2-A)
- Q1 pad 4: Net-(Q1-G) -> Net-(D2-K)
- Q2 pad 4: Net-(Q2-G) -> Net-(D3-K)
- Q2 pad 5: Net-(M1-A) -> Net-(D2-A)
- Q3 pad 1: Net-(M1-B) -> Net-(D4-A)
- Q3 pad 2: Net-(M1-B) -> Net-(D4-A)
- Q3 pad 3: Net-(M1-B) -> Net-(D4-A)
- Q4 pad 5: Net-(M1-B) -> Net-(D4-A)
- Q5 pad 1: Net-(M1-C) -> Net-(D6-A)
- Q5 pad 2: Net-(M1-C) -> Net-(D6-A)
- Q5 pad 3: Net-(M1-C) -> Net-(D6-A)
- Q6 pad 5: Net-(M1-C) -> Net-(D6-A)
- R1 pad 1: +5V -> +3.3V
- R1 pad 2: Net-(U2-FB) -> Net-(U1-SDA)
- R10 pad 1: Net-(U3-GLC) -> Net-(U2-GLC)
- R11 pad 1: /7SA -> +5V
- R11 pad 2: Net-(U6-A) -> Net-(U4-FB)
- R12 pad 1: /7SB -> +12V
- R12 pad 2: Net-(U6-B) -> Net-(U4-EN)
- R13 pad 1: /7SC -> Net-(U4-FB)
- R13 pad 2: Net-(U6-C) -> GND
- R2 pad 1: Net-(U2-FB) -> +3.3V
- R2 pad 2: GND -> Net-(U1-SCL)
- R3 pad 1: +3.3V -> Net-(U2-GHA)
- R3 pad 2: Net-(R3-Pad2) -> Net-(D2-K)
- R4 pad 1: Net-(R3-Pad2) -> Net-(U2-GLA)
- R4 pad 2: Net-(U1-GPIO8/ADC1_CH7) -> Net-(D3-K)
- R5 pad 1: Net-(U3-GHA) -> +3.3V
- R5 pad 2: Net-(Q1-G) -> Net-(R5-Pad2)
- R6 pad 1: Net-(U3-GLA) -> Net-(R5-Pad2)
- R6 pad 2: Net-(Q2-G) -> Net-(U3-GPIO8/ADC1_CH7)
- R7 pad 1: Net-(U3-GHB) -> Net-(U2-GHB)
- R8 pad 1: Net-(U3-GLB) -> Net-(U2-GLB)
- R9 pad 1: Net-(U3-GHC) -> Net-(U2-GHC)
- SW1 pad 1: Net-(R3-Pad2) -> Net-(R5-Pad2)
- U1 pad 10: unconnected-(U1-GPIO17/ADC2_CH6-Pad10) -> GND
- U1 pad 2: +3.3V -> Net-(U1-SCL)
- U1 pad 3: unconnected-(U1-CHIP_PU-Pad3) -> Net-(U1-SDA)
- U1 pad 4: Net-(U1-GPIO4/ADC1_CH3) -> GND
- U1 pad 5: Net-(J1-Pin_4) -> +3.3V
- U1 pad 6: Net-(J1-Pin_3) -> Net-(U1-VOUT)
- U1 pad 7: Net-(J1-Pin_2) -> Net-(U1-C1+)
- U1 pad 8: unconnected-(U1-GPIO15/ADC2_CH4/32K_P-Pad8) -> Net-(U1-C1-)
- U1 pad 9: unconnected-(U1-GPIO16/ADC2_CH5/32K_N-Pad9) -> +3.3V
- U2 pad 1: GND -> /INHA
- U2 pad 2: Net-(U2-SW) -> /INHB
- U2 pad 3: +12V -> /INHC
- U2 pad 4: Net-(U2-FB) -> /INLA
- U2 pad 5: unconnected-(U2-EN-Pad5) -> /INLB
- U2 pad 6: Net-(U2-BST) -> /INLC
- U3 pad 1: /INHA -> +3.3V
- U3 pad 10: Net-(U3-GLB) -> unconnected-(U3-GPIO17/ADC2_CH6-Pad10)
- U3 pad 11: Net-(U3-GLA) -> unconnected-(U3-GPIO18/ADC2_CH7-Pad11)
- U3 pad 12: Net-(M1-C) -> Net-(U3-GPIO8/ADC1_CH7)
- U3 pad 13: Net-(U3-GHC) -> unconnected-(U3-GPIO3/ADC1_CH2-Pad13)
- U3 pad 14: Net-(U3-BSTC) -> unconnected-(U3-GPIO46-Pad14)
- U3 pad 15: Net-(M1-B) -> /INLC
- U3 pad 16: Net-(U3-GHB) -> /INLB
- U3 pad 17: Net-(U3-BSTB) -> /INLA
- U3 pad 18: Net-(M1-A) -> /INHC
- U3 pad 19: Net-(U3-GHA) -> /INHB
- U3 pad 2: /INHB -> +3.3V
- U3 pad 20: Net-(U3-BSTA) -> /INHA
- U3 pad 3: /INHC -> unconnected-(U3-CHIP_PU-Pad3)
- U3 pad 4: /INLA -> unconnected-(U3-GPIO4/ADC1_CH3-Pad4)
- U3 pad 5: /INLB -> Net-(J1-Pin_4)
- U3 pad 6: /INLC -> Net-(J1-Pin_3)
- U3 pad 7: +12V -> Net-(J1-Pin_2)
- U3 pad 8: GND -> unconnected-(U3-GPIO15/ADC2_CH4/32K_P-Pad8)
- U3 pad 9: Net-(U3-GLC) -> unconnected-(U3-GPIO16/ADC2_CH5/32K_N-Pad9)
- U4 pad 1: /7SC -> GND
- U4 pad 2: /7SDP -> Net-(U4-SW)
- U4 pad 3: /7SD -> +12V
- U4 pad 4: /7SE -> Net-(U4-FB)
- U4 pad 5: /7S3 -> Net-(U4-EN)
- U4 pad 6: /7S2 -> Net-(U4-BST)
Routing:
- net Net-(U3-GPIO8/ADC1_CH7): track 0.00 -> 92.4 mm
- net Net-(U1-GPIO8/ADC1_CH7): track 90.5 -> 0.00 mm
- net +3.3V: track 138.7 -> 206.9 mm, vias 3 -> 0
- net Net-(U6-B): track 68.0 -> 0.00 mm
- net Net-(U6-F): track 67.7 -> 0.00 mm
- net Net-(U6-A): track 66.7 -> 0.00 mm, vias 1 -> 0
- net Net-(U1-GPIO4/ADC1_CH3): track 53.7 -> 0.00 mm
- net Net-(U6-D): track 53.0 -> 0.00 mm, vias 1 -> 0
- net Net-(U1-SCL): track 0.00 -> 52.5 mm
- net Net-(U6-E): track 52.1 -> 0.00 mm, vias 1 -> 0
- net Net-(U1-SDA): track 0.00 -> 49.4 mm
- net Net-(U1-GPIO2/ADC1_CH1): track 47.3 -> 0.00 mm, vias 2 -> 0
- net Net-(U1-GPIO1/ADC1_CH0): track 45.3 -> 0.00 mm, vias 2 -> 0
- net Net-(U6-G): track 44.8 -> 0.00 mm, vias 1 -> 0
- net Net-(U6-DP): track 44.8 -> 0.00 mm, vias 1 -> 0
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- added copper zone on F.Cu, net Net-(D2-A)
- added copper zone on F.Cu, net Net-(D4-A)
- added copper zone on F.Cu, net Net-(D6-A)
- removed copper zone on F.Cu, net Net-(M1-A)
- removed copper zone on B.Cu, net Net-(M1-B)
- removed copper zone on F.Cu, net Net-(M1-B)
- removed copper zone on F.Cu, net Net-(M1-C)
Other:
- board size 150 x 100 mm -> 150 x 110 mm
- board text added: "Spin Coater Prototype 2026 v2"
- board text removed: "Spin Coater Prototype 2025"

Commit message: Replace gate driver decoupling capacitor
Parts:
- added C15: 10uF, Capacitor_SMD:C_1206_3216Metric, F.Cu at (98.8, 124.2)
- C14: value 22uF -> 10uF; footprint Capacitor_SMD:C_1210_3225Metric -> Capacitor_SMD:C_1206_3216Metric
- R11: value 24k -> 22k
- renumbered C15 to C16, C16 to C17, C17 to C18, C18 to C19, C19 to C20, D9 to D5, D5 to D6, D6 to D7, D7 to D8, D8 to D9
Routing:
- net +12V: track 55.5 -> 58.0 mm
- net GND: vias 294 -> 292

Commit message: Renumber
Parts:
- renumbered D6 to D5, D7 to D6, D8 to D7, D9 to D8, D5 to D9
Routing:
- net GND: vias 292 -> 297
